Commit message: EKF working and lidar package is there.

File: tinycar_description/urdf/controllers/tinycar.gazebo.xacro (robot description, xacro)
@@ -29,3 +29,73 @@
     <plugin name="gz::sim::systems::Imu" filename="gz-sim-imu-system"/>
   </gazebo>
+    <!-- IMU attached to imu_link -->
+    <gazebo reference="imu_link">
+        <sensor name="imu_sensor" type="imu">
+            <frame_id>imu_link</frame_id>
+            <always_on>true</always_on>
+            <update_rate>100</update_rate>
+            <topic>/imu</topic>
+            <imu>
+            <angular_velocity><!-- Optional: a simple visual/collision so you can see it in RViz/Gazebo -->
+    <link name="imu_link_visual">
+      <visual>
+        <origin xyz="0 0 0" rpy="0 0 0"/>
+        <geometry><box size="0.03 0.02 0.01"/></geometry>
+      </visual>
+      <collision>
+        <origin xyz="0 0 0" rpy="0 0 0"/>
+        <geometry><box size="0.03 0.02 0.01"/></geometry>
+      </collision>
+      <inertial>
+        <origin xyz="0 0 0" rpy="0 0 0"/>
+        <mass value="0.02"/>
+        <inertia ixx="1e-6" iyy="1e-6" izz="1e-6" ixy="0" ixz="0" iyz="0"/>
+      </inertial>
+    </link>
+    <joint name="imu_visual_joint" type="fixed">
+      <origin xyz="0 0 0" rpy="0 0 0"/>
+      <parent link="imu_link"/>
+      <child link="imu_link_visual"/>
+    </joint>
+                <x><noise type="gaussian"><mean>0</mean><stddev>0.001</stddev></noise></x>
+                <y><noise type="gaussian"><mean>0</mean><stddev>0.001</stddev></noise></y>
+                <z><noise type="gaussian"><mean>0</mean><stddev>0.001</stddev></noise></z>
+            </angular_velocity>
+            <linear_acceleration>
+                <x><noise type="gaussian"><mean>0</mean><stddev>0.01</stddev></noise></x>
+                <y><noise type="gaussian"><mean>0</mean><stddev>0.01</stddev></noise></y>
+                <z><noise type="gaussian"><mean>0</mean><stddev>0.01</stddev></noise></z>
+            </linear_acceleration>
+            </imu>
+        </sensor>
+    </gazebo>
+      <!-- LiDAR attached to base_laser -->
+  <gazebo reference="base_laser">
+    <sensor name="gpu_lidar" type="gpu_lidar">
+      <topic>/scan</topic>
+      <update_rate>20</update_rate>
+      <always_on>true</always_on>
+      <visualize>true</visualize>
+      <lidar>
+        <scan>
+          <horizontal>
+            <samples>720</samples>
+            <resolution>1</resolution>
+            <min_angle>-3.14159</min_angle>
+            <max_angle>3.14159</max_angle>
+          </horizontal>
+        </scan>
+        <range>
+          <min>0.05</min>
+          <max>12.0</max>
+          <resolution>0.01</resolution>
+        </range>
+        <noise>
+          <type>gaussian</type>
+          <mean>0.0</mean>
+          <stddev>0.01</stddev>
+        </noise>
+      </lidar>
+    </sensor>
+  </gazebo>
 </robot>

File: tinycar_description/urdf/tinycar.urdf.xacro (robot description, xacro)
@@ -4,4 +4,5 @@
   <xacro:include filename="$(find tinycar_description)/urdf/controllers/tinycar.ros2_control.xacro"/>
   <xacro:include filename="$(find tinycar_description)/urdf/controllers/tinycar.gazebo.xacro"/>
+<xacro:include filename="$(find tinycar_description)/urdf/sensors/tinycar.sensors.xacro"/>
     <link name="base_footprint" />
     <link name="base_link">
@@ -131,3 +132,4 @@
         <origin xyz="0.045 0.0 -0.0265" rpy="0 0 0" />
     </joint>
+    <xacro:agribot_sensors/>
 </robot>
