Commit message: Changed inertial to for collision and  made tinymanual changed.

File: tinycar_description/urdf/tinycar.urdf.xacro (robot description, xacro)
@@ -21,15 +21,13 @@
     <inertial>
         <mass value="2.768772"/>
-        <!-- Converted mm → m -->
-        <origin xyz="-0.028754 0.002600 -0.011369" rpy="0 0 0"/>
-        <!-- Converted kg·mm² → kg·m² -->
+        <origin xyz="-0.01 0 0.00861" rpy="0 0 0"/>
         <inertia
-            ixx="0.0046876"
-            ixy="-0.00002531"
-            ixz="-0.00082487"
-            iyy="0.0069378"
-            iyz="-0.00017317"
-            izz="0.0075916"/>
-    </inertial>
+            ixx="0.00455"
+            iyy="0.00826"
+            izz="0.00833"
+            ixy="0.0"
+            ixz="0.0"
+            iyz="0.0"/>
+        </inertial>
     </link>
     <link name="left_wheel">
@@ -48,13 +46,13 @@
         </collision>
          <inertial>
-        <mass value="0.017054"/>
-        <origin xyz="-0.00000653 -0.009275 0.00000035" rpy="0 0 0"/>
-        <inertia
-            ixx="0.0000024304"
-            ixy="0.0"
-            ixz="-0.00000000036"
-            iyy="0.0000039401"
-            iyz="0.0"
-            izz="0.0000024304"/>
+            <mass value="0.017054"/>
+            <origin xyz="0 0 0" rpy="0 0 0"/>
+            <inertia
+                ixx="0.00000273"
+                iyy="0.00000432"
+                izz="0.00000273"
+                ixy="0.0"
+                ixz="0.0"
+                iyz="0.0"/>
     </inertial>
     </link>
@@ -73,14 +71,14 @@
             </geometry>
         </collision>
-        <inertial>
+      <inertial>
         <mass value="0.017054"/>
-        <origin xyz="-0.00000653 -0.009275 0.00000035" rpy="0 0 0"/>
+        <origin xyz="0 0 0" rpy="0 0 0"/>
         <inertia
-            ixx="0.0000024304"
+            ixx="0.00000273"
+            iyy="0.00000432"
+            izz="0.00000273"
             ixy="0.0"
-            ixz="-0.00000000036"
-            iyy="0.0000039401"
-            iyz="0.0"
-            izz="0.0000024304"/>
+            ixz="0.0"
+            iyz="0.0"/>
     </inertial>
     </link>
@@ -100,14 +98,14 @@
         </collision>
     <inertial>
-        <mass value="0.009834"/>
-        <origin xyz="0.0 0.0 -0.013911" rpy="0 0 0"/>
-        <inertia
-            ixx="0.0000008909"
-            ixy="0.0"
-            ixz="0.0"
-            iyy="0.0000008909"
-            iyz="0.0"
-            izz="0.0000010717"/>
-    </inertial>
+    <mass value="0.009834"/>
+    <origin xyz="0 0 -0.005" rpy="0 0 0"/>
+    <inertia
+        ixx="0.00000246"
+        iyy="0.00000246"
+        izz="0.00000246"
+        ixy="0.0"
+        ixz="0.0"
+        iyz="0.0"/>
+</inertial>
     </link>
     <joint name="virtual_joint" type="fixed">
@@ -131,5 +129,5 @@
         <parent link="base_link"/>
         <child link="caster_wheel"/>
-        <origin xyz="0.035 0.0 -0.0265" rpy="0 0 0" />
+        <origin xyz="0.045 0.0 -0.0265" rpy="0 0 0" />
     </joint>
 </robot>

Commit message: tried ros2_control

File: tinycar_description/urdf/tinycar.urdf.xacro (robot description, xacro)
@@ -22,5 +22,5 @@
     <inertial>
         <mass value="2.768772"/>
-        <origin xyz="-0.01 0 0.00861" rpy="0 0 0"/>
+        <origin xyz="-0.02 0 0.00561" rpy="0 0 0"/>
         <inertia
             ixx="0.00455"
